File: fortissimo-ii.kicad_sch (KiCad schematic)
At the start: 0 parts

Commit message: created schematic v1
Parts:
- added 0.1uF1, 0.1uF2: USB_C_Plug_USB2.0, Connector_USB:USB_C_Receptacle_JAE_DX07S016JA1R1500, symbol Connector:USB_C_Plug_USB2.0
- added Brd1: SSD1306, SSD1306:128x64OLED, symbol SSD1306-128x64_OLED:SSD1306
- added C1, C10, C2, C3, C4: 10uF, symbol Device:C
- added C11, C14, C17, C20, C23: 100uF, symbol Device:C
- added C12, C13, C15, C16, C18, C19, C21, C22, C24, C25: 4.7nF, symbol Device:C
- added C5: 0.1uF, symbol Device:C
- added D1, D10, D11, D12, D13, D14, D15, D16, D17, D18, D19, D2, D20, D21, D22, D23, D24, D25, D26, D27, D28, D29, D3, D30, D31, D32, D33, D34, D4, D5, D6, D7, D8, D9: D, symbol Device:D
- added D35, D36, D37, D38, D74: D_Schottky 100uF, Diode_SMD:D_SMA, symbol Device:D_Schottky
- added D39, D40, D41, D42, D43, D44, D45, D46, D47, D48, D49, D50, D51, D52, D53, D54, D55, D56, D57, D58, D59, D60, D61, D62, D63, D64, D65, D66, D67, D68, D69, D70, D71, D72, D73: SK6812MINI, LED_SMD:LED_SK6812MINI_PLCC4_3.5x3.5mm_P1.75mm, symbol LED:SK6812MINI
- added FB1: FerriteBead, Ferrite_THT:LairdTech_28C0236-0JW-10, symbol Device:FerriteBead
- added J1, J2: USB_A, Connector_USB:USB3_A_Molex_48393-001, symbol Connector:USB_A
- added R1: 2.7k, symbol Device:R
- added R6, R7: 5.1k, symbol Device:R
- added SW1, SW10, SW11, SW12, SW13, SW14, SW15, SW16, SW17, SW18, SW19, SW2, SW20, SW21, SW22, SW23, SW24, SW25, SW26, SW27, SW28, SW29, SW3, SW30, SW31, SW32, SW33, SW34, SW4, SW5, SW6, SW7, SW8, SW9: SW_Push, symbol Switch:SW_Push
- added SW35: RotaryEncoder_Switch, symbol Device:RotaryEncoder_Switch
- added SW36: LANG_SWITCH, symbol Switch:SW_Push
- added SW_BOOTSEL1: BOOTSEL_SWITCH, symbol Switch:SW_Push
- added U1: ~, PGA2040:PGA2040, symbol PGA2040:PGA2040
- added U2: FE1.1s, Package_SO:SSOP-28_3.9x9.9mm_P0.635mm, symbol Interface_USB:FE1.1s
- added U3: USBLC6-2SC6, Package_TO_SOT_SMD:SOT-23-6, symbol Power_Protection:USBLC6-2SC6
- added Y1: 12MHz Crystal, symbol Device:Crystal
Connections:
- new net: D56.1 (DOUT), D57.3 (DIN)
- new net: D55.1 (DOUT), D56.3 (DIN)
- new net: D71.1 (DOUT), D72.3 (DIN)
- new net: D70.1 (DOUT), D71.3 (DIN)
- new net: D3.2 (A), SW3.2
- new net: D39.3 (DIN), D40.1 (DOUT)
- new net: D40.3 (DIN), D41.1 (DOUT)
- new net: D14.2 (A), SW14.2
- new net: D9.2 (A), SW9.2
- new net: 0.1uF1.A4 (VBUS), 0.1uF1.A9 (VBUS), 0.1uF1.B4 (VBUS), 0.1uF1.B9 (VBUS), C4.2, D38.1 (K)
- new net: D29.2 (A), SW29.2
- new net: C10.2, D74.1 (K), U2.18 (VBUSM), U2.20 (VDD5)
- new net: D18.2 (A), SW18.2
- new net: D8.2 (A), SW8.2
- new net: D19.2 (A), SW19.2
- new net: D65.1 (DOUT), D66.3 (DIN)
- new net: D64.1 (DOUT), D65.3 (DIN)
- new net: D63.1 (DOUT), D64.3 (DIN)
- new net: D62.1 (DOUT), D63.3 (DIN)
- new net: D53.3 (DIN), D66.1 (DOUT)
- new net: 0.1uF1.A5 (CC), R7.1
- new net: 0.1uF1.A6 (D+), U2.7 (DP3)
- new net: 0.1uF1.A7 (D-), U2.6 (DM3)
- new net: D7.2 (A), SW7.2
- new net: D10.2 (A), SW10.2
- new net: D69.1 (DOUT), D70.3 (DIN)
- new net: D68.1 (DOUT), D69.3 (DIN)
- new net: D22.2 (A), SW22.2
- new net: D25.2 (A), SW25.2
- new net: D54.1 (DOUT), D55.3 (DIN)
- new net: D6.2 (A), SW6.2
- new net: D12.2 (A), SW12.2
- new net: 0.1uF2.A4 (VBUS), 0.1uF2.A9 (VBUS), 0.1uF2.B4 (VBUS), 0.1uF2.B9 (VBUS), D35.2 (A)
- new net: 0.1uF2.A5 (CC), R6.1
- new net: 0.1uF2.A6 (D+), U3.3 (I/O2)
- new net: 0.1uF2.A7 (D-), U3.1 (I/O1)
- new net: D5.2 (A), SW5.2
- new net: D50.1 (DOUT), D51.3 (DIN)
- new net: D49.1 (DOUT), D50.3 (DIN)
- new net: D30.2 (A), SW30.2
- new net: SW_BOOTSEL1.2, U1.A7 (BOOTSEL)
- new net: D4.2 (A), SW4.2
- new net: D27.2 (A), SW27.2
- new net: D1.2 (A), SW1.2
- new net: D67.1 (DOUT), D68.3 (DIN)
- new net: D2.2 (A), SW2.2
- new net: R1.2, U2.14 (REXT)
- new net: D57.1 (DOUT), D58.3 (DIN)
- new net: D35.1 (K), FB1.1
- new net: U2.15 (DMU), U3.4 (I/O2)
- new net: U2.16 (DPU), U3.6 (I/O1)
- new net: D58.1 (DOUT), D59.3 (DIN)
- new net: D11.2 (A), SW11.2
- new net: D45.3 (DIN), D52.1 (DOUT)
- new net: D51.1 (DOUT), D52.3 (DIN)
- new net: D21.2 (A), SW21.2
- new net: D34.2 (A), SW34.2
- new net: D43.3 (DIN), D44.1 (DOUT)
- new net: D44.3 (DIN), D45.1 (DOUT)
- new net: C3.2, D36.1 (K), J1.1 (VBUS)
- new net: D17.2 (A), SW17.2
- new net: C2.2, D37.1 (K), J2.1 (VBUS)
- new net: D24.2 (A), SW24.2
- new net: D48.1 (DOUT), D49.3 (DIN)
- new net: D32.2 (A), SW32.2
- new net: D42.3 (DIN), D43.1 (DOUT)
- new net: J1.2 (D-), U2.10 (DM1)
- new net: J1.3 (D+), U2.11 (DP1)
- new net: D72.1 (DOUT), D73.3 (DIN)
- new net: D41.3 (DIN), D42.1 (DOUT)
- new net: D13.2 (A), SW13.2
- new net: D20.2 (A), SW20.2
- new net: D28.2 (A), SW28.2
- new net: D53.1 (DOUT), D54.3 (DIN)
- new net: D46.3 (DIN), D59.1 (DOUT)
- new net: U2.3 (XIN), Y1.1
- new net: U2.2 (XOUT), Y1.2
- new net: D33.2 (A), SW33.2
- new net: D47.1 (DOUT), D48.3 (DIN)
- new net: D16.2 (A), SW16.2
- new net: D61.1 (DOUT), D62.3 (DIN)
- new net: J2.2 (D-), U2.8 (DM2)
- new net: J2.3 (D+), U2.9 (DP2)
- new net: D46.1 (DOUT), D47.3 (DIN)
- new net: D60.1 (DOUT), D61.3 (DIN)
- new net: D60.3 (DIN), D73.1 (DOUT)
- new net: D31.2 (A), SW31.2
- new net: Brd1.3 (SCL), U1.C8 (GPIO27/ADC1)
- new net: Brd1.4 (SDA), U1.D7 (GPIO26/ADC0)
- new net: D26.2 (A), SW26.2
- new net: D15.2 (A), SW15.2
- new net: D23.2 (A), SW23.2
- new net +3.3V: U1.B3 (3V3)
- new net +3V3: C5.1, U2.13 (VD33)
- new net GND: 0.1uF1.A1 (GND), 0.1uF1.A12 (GND), 0.1uF1.B1 (GND), 0.1uF1.B12 (GND), 0.1uF1.S1 (SHIELD), 0.1uF2.A1 (GND), 0.1uF2.A12 (GND), 0.1uF2.B1 (GND), 0.1uF2.B12 (GND), 0.1uF2.S1 (SHIELD), Brd1.1 (GND), C1.1, C10.1, C11.1, C12.1, C13.1, C14.1, C15.1, C16.1, C17.1, C18.1, C19.1, C2.1, C20.1, C21.1, C22.1, C23.1, C24.1, C25.1, C3.1, C4.1, C5.2, D60.2 (VSS), D61.2 (VSS), D62.2 (VSS), D63.2 (VSS), D64.2 (VSS), D65.2 (VSS), D66.2 (VSS), D67.2 (VSS), D68.2 (VSS), D69.2 (VSS), D70.2 (VSS), D71.2 (VSS), D72.2 (VSS), D73.2 (VSS), J1.4 (GND), J1.5 (Shield), J2.4 (GND), J2.5 (Shield), R1.1, R6.2, R7.2, SW36.2, SW_BOOTSEL1.1, U1.GND, U2.1 (VSS), U2.27 (TESTJ/EESDA), U3.2 (GND)
- new net LANG: SW36.1, U1.D8 (GPIO25)
- new net MCU-D+: U1.A5 (USB_DP), U2.5 (DP4)
- new net MCU-D-: U1.A6 (USB_DM), U2.4 (DM4)
- new net VBUS: Brd1.2 (VCC), C1.2, C11.2, C12.2, C13.2, C14.2, C15.2, C16.2, C17.2, C18.2, C19.2, C20.2, C21.2, C22.2, C23.2, C24.2, C25.2, D36.2 (A), D37.2 (A), D38.2 (A), D39.4 (VDD), D40.4 (VDD), D41.4 (VDD), D42.4 (VDD), D43.4 (VDD), D44.4 (VDD), D45.4 (VDD), D46.4 (VDD), D47.4 (VDD), D48.4 (VDD), D49.4 (VDD), D50.4 (VDD), D51.4 (VDD), D52.4 (VDD), D53.4 (VDD), D54.4 (VDD), D55.4 (VDD), D56.4 (VDD), D57.4 (VDD), D58.4 (VDD), D59.4 (VDD), D60.4 (VDD), D61.4 (VDD), D62.4 (VDD), D63.4 (VDD), D64.4 (VDD), D65.4 (VDD), D66.4 (VDD), D67.4 (VDD), D68.4 (VDD), D69.4 (VDD), D70.4 (VDD), D71.4 (VDD), D72.4 (VDD), D73.4 (VDD), D74.2 (A), FB1.2, U1.A2 (VBUS), U3.5 (VBUS)
- new net col1: SW1.1, SW15.1, SW22.1, SW29.1, SW8.1, U1.H4 (GPIO13)
- new net col2: SW16.1, SW2.1, SW23.1, SW30.1, SW9.1, U1.G4 (GPIO14)
- new net col3: SW10.1, SW17.1, SW24.1, SW3.1, SW31.1, U1.H5 (GPIO15)
- new net col4: SW11.1, SW18.1, SW25.1, SW32.1, SW4.1, U1.G5 (GPIO16)
- new net col5: SW12.1, SW19.1, SW26.1, SW33.1, SW5.1, U1.H6 (GPIO17)
- new net col6: SW13.1, SW20.1, SW27.1, SW34.1, SW6.1, U1.G6 (GPIO18)
- new net col7: SW14.1, SW21.1, SW28.1, SW7.1, U1.H7 (GPIO19)
- new net row1: D1.1 (K), D2.1 (K), D3.1 (K), D4.1 (K), D5.1 (K), D6.1 (K), D7.1 (K), U1.G8 (GPIO20)
- new net row2: D10.1 (K), D11.1 (K), D12.1 (K), D13.1 (K), D14.1 (K), D8.1 (K), D9.1 (K), U1.F8 (GPIO21)
- new net row3: D15.1 (K), D16.1 (K), D17.1 (K), D18.1 (K), D19.1 (K), D20.1 (K), D21.1 (K), U1.F7 (GPIO22)
- new net row4: D22.1 (K), D23.1 (K), D24.1 (K), D25.1 (K), D26.1 (K), D27.1 (K), D28.1 (K), U1.E8 (GPIO23)
- new net row5: D29.1 (K), D30.1 (K), D31.1 (K), D32.1 (K), D33.1 (K), D34.1 (K), U1.E7 (GPIO24)
- no-connect marks 0 -> 12
