File: fortissimo-ii.kicad_sch (KiCad schematic)
At the start: 146 parts, among them J1 USB_A, J2 USB_A, SW1 SW_Push, SW10 SW_Push, SW11 SW_Push, SW12 SW_Push, SW13 SW_Push, SW14 SW_Push, SW15 SW_Push, SW16 SW_Push, SW17 SW_Push, SW18 SW_Push, SW19 SW_Push, SW2 SW_Push, SW20 SW_Push, SW21 SW_Push, SW22 SW_Push, SW23 SW_Push, SW24 SW_Push, SW25 SW_Push, SW26 SW_Push, SW27 SW_Push, SW28 SW_Push, SW29 SW_Push, SW3 SW_Push, SW30 SW_Push, SW31 SW_Push, SW32 SW_Push, SW33 SW_Push, SW34 SW_Push, SW35 RotaryEncoder_Switch, SW36 LANG_SWITCH, SW4 SW_Push, SW5 SW_Push, SW6 SW_Push, SW7 SW_Push, SW8 SW_Push, SW9 SW_Push, U2 FE1.1s, U3 USBLC6-2SC6, Y1 12MHz Crystal

Commit message: changes from jul 29
Parts:
- removed 0.1uF1, 0.1uF2: USB_C_Plug_USB2.0, Connector_USB:USB_C_Receptacle_JAE_DX07S016JA1R1500, symbol Connector:USB_C_Plug_USB2.0
- removed C1, C10, C2, C3, C4, C6: 10uF, Capacitor_SMD:C_0805_2012Metric, symbol Device:C
- removed C11, C14, C17, C20, C23: 100uF, Capacitor_SMD:C_0805_2012Metric, symbol Device:C
- removed C12, C13, C15, C16, C18, C19, C21, C22, C24, C25: 4.7nF, Capacitor_SMD:C_0805_2012Metric, symbol Device:C
- removed C5: 0.1uF, Capacitor_SMD:C_0805_2012Metric, symbol Device:C
- removed D35, D36, D37, D38, D74: D_Schottky 100uF, Capacitor_THT:C_Radial_D5.0mm_H11.0mm_P2.00mm, symbol Device:D_Schottky
- removed D39, D40, D41, D42, D43, D44, D45, D46, D47, D48, D49, D50, D51, D52, D53, D54, D55, D56, D57, D58, D59, D60, D61, D62, D63, D64, D65, D66, D67, D68, D69, D70, D71, D72, D73: SK6812MINI, Keebio-Parts:SK6812-MINI-E, symbol LED:SK6812MINI
- removed FB1: FerriteBead, Inductor_SMD:L_0805_2012Metric, symbol Device:FerriteBead
- removed J1, J2: USB_A, Connector_USB:USB_A_Receptacle_GCT_USB1046, symbol Connector:USB_A
- removed R6, R7: 5.1k, Resistor_SMD:R_0805_2012Metric, symbol Device:R
- removed SW1, SW10, SW11, SW12, SW13, SW14, SW15, SW16, SW17, SW18, SW19, SW2, SW20, SW21, SW22, SW23, SW24, SW25, SW26, SW27, SW28, SW29, SW3, SW30, SW31, SW32, SW33, SW34, SW4, SW5, SW6, SW7, SW8, SW9: SW_Push, Keebio-Parts:MX-Alps-Choc-1U, symbol Switch:SW_Push
- removed SW35: RotaryEncoder_Switch, Rotary_Encoder:RotaryEncoder_Alps_EC11E-Switch_Vertical_H20mm_CircularMountingHoles, symbol Device:RotaryEncoder_Switch
- removed SW36: LANG_SWITCH, Button_Switch_THT:SW_PUSH_6mm, symbol Switch:SW_Push
- removed SW_BOOTSEL1: BOOTSEL_SWITCH, Button_Switch_THT:SW_PUSH_6mm, symbol Switch:SW_Push
- removed U1: ~, PGA2040:PGA2040, symbol PGA2040:PGA2040
- removed U2: FE1.1s, Package_SO:SSOP-28_3.9x9.9mm_P0.635mm, symbol Interface_USB:FE1.1s
- removed U3: USBLC6-2SC6, Package_TO_SOT_SMD:SOT-23-6, symbol Power_Protection:USBLC6-2SC6
- removed Y1: 12MHz Crystal, Crystal:Crystal_SMD_3225-4Pin_3.2x2.5mm_HandSoldering, symbol Device:Crystal
- added A1, A2: RaspberryPi_Pico, Module:RaspberryPi_Pico_Common_Unspecified, symbol MCU_Module:RaspberryPi_Pico
- added Brd2: SSD1306, SSD1306:128x64OLED, symbol SSD1306-128x64_OLED:SSD1306
- added D35, D36, D37, D72, D73, D74: PESD5V0S1UL, Diode_SMD:D_SOD-882, symbol Diode:PESD5V0S1UL
- added D38, D39, D40, D41, D42, D43, D44, D45, D46, D47, D48, D49, D50, D51, D52, D53, D54, D55, D56, D57, D58, D59, D60, D61, D62, D63, D64, D65, D66, D67, D68, D69, D70, D71: D, Diode_THT:D_DO-35_SOD27_P7.62mm_Horizontal, symbol Device:D
- added J1, J2: AudioJack4, Keebio-Parts:TRRS-PJ-320A, symbol Connector_Audio:AudioJack4
- added R2, R3, R4: 4.7k, Resistor_SMD:R_0603_1608Metric, symbol Device:R
- added SW1, SW10, SW11, SW12, SW13, SW14, SW15, SW16, SW17, SW18, SW19, SW2, SW20, SW21, SW22, SW23, SW24, SW25, SW26, SW27, SW28, SW29, SW3, SW30, SW31, SW32, SW33, SW36, SW37, SW38, SW39, SW4, SW41, SW42, SW43, SW44, SW45, SW46, SW47, SW48, SW49, SW5, SW50, SW51, SW52, SW53, SW54, SW55, SW56, SW57, SW58, SW59, SW6, SW60, SW61, SW62, SW63, SW64, SW65, SW66, SW67, SW68, SW69, SW7, SW8, SW9: SW_Push_45deg, Keebio-Parts:Low-Profile-Choc-MX, symbol Switch:SW_Push_45deg
- added SW34, SW40: SW_Push_45deg, Keebio-Parts:MX-Alps-Choc-2U-StabFlip, symbol Switch:SW_Push_45deg
- added SW35: LANG, Button_Switch_THT:SW_PUSH_6mm, symbol Switch:SW_Push
- R1: value 2.7k -> 4.7k; footprint Resistor_SMD:R_0805_2012Metric -> Resistor_SMD:R_0603_1608Metric
Connections:
- net +3.3V is gone; now on net VBUS: Brd1.2 (VCC)
- net GND: now also A1.13 (GND), A1.18 (GND), A1.23 (GND), A1.28 (GND), A1.3 (GND), A1.38 (GND), A1.8 (GND), A2.13 (GND), A2.18 (GND), A2.23 (GND), A2.28 (GND), A2.3 (GND), A2.38 (GND), A2.8 (GND), Brd2.1 (GND), D35.1 (K), D36.1 (K), D37.1 (K), D72.1 (K), D73.1 (K), D74.1 (K), J1.T, J2.T, SW35.2; no longer R1.1
- net VBUS: now also R1.1, A1.40 (VBUS), A2.40 (VBUS), Brd2.2 (VCC), D35.2 (A), D72.2 (A), J1.S, J2.S, R2.1, R3.1, R4.1
- net at D3.2 (A): now also SW3.2
- net at D14.2 (A): now also SW14.2
- net at D9.2 (A): now also SW9.2
- net at D29.2 (A): now also SW29.2
- net at D18.2 (A): now also SW18.2
- net at D8.2 (A): now also SW8.2
- net at D19.2 (A): now also SW19.2
- net at D7.2 (A): now also SW7.2
- net at D10.2 (A): now also SW10.2
- net at D22.2 (A): now also SW22.2
- net at D25.2 (A): now also SW25.2
- net at D6.2 (A): now also SW6.2
- net at D12.2 (A): now also SW12.2
- net at D5.2 (A): now also SW5.2
- net at D30.2 (A): now also SW30.2
- net at D4.2 (A): now also SW4.2
- net at D27.2 (A): now also SW27.2
- net at D1.2 (A): now also SW1.2
- net at D2.2 (A): now also SW2.2
- net L_SDA: now reaches R1.2
- net L_SDA: now also Brd1.4 (SDA), A1.34 (GPIO28_ADC2), D36.2 (A), J1.R2
- net at D11.2 (A): now also SW11.2
- net at D21.2 (A): now also SW21.2
- net at D34.2 (A): now also SW34.2
- net at D17.2 (A): now also SW17.2
- net at D24.2 (A): now also SW24.2
- net at D32.2 (A): now also SW32.2
- net at D13.2 (A): now also SW13.2
- net at D20.2 (A): now also SW20.2
- net at D28.2 (A): now also SW28.2
- net at D33.2 (A): now also SW33.2
- net at D16.2 (A): now also SW16.2
- net at D31.2 (A): now also SW31.2
- net L_SCL: now reaches Brd1.3 (SCL)
- net L_SCL: now also A1.32 (GPIO27_ADC1), D37.2 (A), J1.R1, R2.2
- net at D26.2 (A): now also SW26.2
- net at D15.2 (A): now also SW15.2
- net at D23.2 (A): now also SW23.2
- net row1 renamed L_row_1
- net L_row_1: now also A1.1 (GPIO0)
- net row2 renamed L_row_2
- net L_row_2: now also A1.2 (GPIO1)
- net row3 renamed L_row_3
- net L_row_3: now also A1.4 (GPIO2)
- net row4 renamed L_row_4
- net L_row_4: now also A1.5 (GPIO3)
- net row5 renamed L_row_5
- net L_row_5: now also A1.6 (GPIO4)
- new net: D67.2 (A), SW65.2
- new net: D48.2 (A), SW46.2
- new net: D51.2 (A), SW49.2
- new net: D38.2 (A), SW36.2
- new net: A1.20 (GPIO15), SW35.1
- new net: D64.2 (A), SW62.2
- new net: D43.2 (A), SW41.2
- new net: D58.2 (A), SW56.2
- new net: D59.2 (A), SW57.2
- new net: D40.2 (A), SW38.2
- new net: D70.2 (A), SW68.2
- new net: D71.2 (A), SW69.2
- new net: D56.2 (A), SW54.2
- new net: D54.2 (A), SW52.2
- new net: D52.2 (A), SW50.2
- new net: D57.2 (A), SW55.2
- new net: D66.2 (A), SW64.2
- new net: D46.2 (A), SW44.2
- new net: D44.2 (A), SW42.2
- new net: D45.2 (A), SW43.2
- new net: D62.2 (A), SW60.2
- new net: D49.2 (A), SW47.2
- new net: D65.2 (A), SW63.2
- new net: D50.2 (A), SW48.2
- new net: D61.2 (A), SW59.2
- new net: D55.2 (A), SW53.2
- new net: D63.2 (A), SW61.2
- new net: D60.2 (A), SW58.2
- new net: D69.2 (A), SW67.2
- new net: D68.2 (A), SW66.2
- new net: D41.2 (A), SW39.2
- new net: D42.2 (A), SW40.2
- new net: D53.2 (A), SW51.2
- new net: D39.2 (A), SW37.2
- new net: D47.2 (A), SW45.2
- new net L_col_1: A1.7 (GPIO5), SW1.1, SW15.1, SW22.1, SW29.1, SW8.1
- new net L_col_2: A1.9 (GPIO6), SW16.1, SW2.1, SW23.1, SW30.1, SW9.1
- new net L_col_3: A1.10 (GPIO7), SW10.1, SW17.1, SW24.1, SW3.1, SW31.1
- new net L_col_4: A1.11 (GPIO8), SW11.1, SW18.1, SW25.1, SW32.1, SW4.1
- new net L_col_5: A1.12 (GPIO9), SW12.1, SW19.1, SW26.1, SW33.1, SW5.1
- new net L_col_6: A1.14 (GPIO10), SW13.1, SW20.1, SW27.1, SW34.1, SW6.1
- new net L_col_7: A1.15 (GPIO11), SW14.1, SW21.1, SW28.1, SW7.1
- new net R_SCL: A2.32 (GPIO27_ADC1), Brd2.3 (SCL), D74.2 (A), J2.R1, R4.2
- new net R_SDA: A2.34 (GPIO28_ADC2), Brd2.4 (SDA), D73.2 (A), J2.R2, R3.2
- new net R_col_1: A2.7 (GPIO5), SW36.1, SW37.1, SW38.1, SW39.1
- new net R_col_2: A2.9 (GPIO6), SW40.1, SW41.1, SW42.1, SW43.1, SW44.1
- new net R_col_3: A2.10 (GPIO7), SW45.1, SW46.1, SW47.1, SW48.1, SW49.1
- new net R_col_4: A2.11 (GPIO8), SW50.1, SW51.1, SW52.1, SW53.1, SW54.1
- new net R_col_5: A2.12 (GPIO9), SW55.1, SW56.1, SW57.1, SW58.1, SW59.1
- new net R_col_6: A2.14 (GPIO10), SW60.1, SW61.1, SW62.1, SW63.1, SW64.1
- new net R_col_7: A2.15 (GPIO11), SW65.1, SW66.1, SW67.1, SW68.1, SW69.1
- new net R_row_1: A2.1 (GPIO0), D38.1 (K), D43.1 (K), D48.1 (K), D53.1 (K), D58.1 (K), D63.1 (K), D68.1 (K)
- new net R_row_2: A2.2 (GPIO1), D39.1 (K), D44.1 (K), D49.1 (K), D54.1 (K), D59.1 (K), D64.1 (K), D69.1 (K)
- new net R_row_3: A2.4 (GPIO2), D40.1 (K), D45.1 (K), D50.1 (K), D55.1 (K), D60.1 (K), D65.1 (K), D70.1 (K)
- new net R_row_4: A2.5 (GPIO3), D41.1 (K), D46.1 (K), D51.1 (K), D56.1 (K), D61.1 (K), D66.1 (K), D71.1 (K)
- new net R_row_5: A2.6 (GPIO4), D42.1 (K), D47.1 (K), D52.1 (K), D57.1 (K), D62.1 (K), D67.1 (K)
- no-connect marks 12 -> 0

Commit message: basically the entire thing
Parts:
- A1, A2: footprint Module:RaspberryPi_Pico_Common_Unspecified -> fortissimo-ii:RaspberryPi_Pico_Common_Unspecified; symbol MCU_Module:RaspberryPi_Pico -> fortissimo:RaspberryPi_Pico
- Brd1, Brd2: footprint SSD1306:128x64OLED -> fortissimo-ii:128x64OLED
- D1, D10, D11, D12, D13, D14, D15, D16, D17, D18, D19, D2, D20, D21, D22, D23, D24, D25, D26, D27, D28, D29, D3, D30, D31, D32, D33, D34, D38, D39, D4, D40, D41, D42, D43, D44, D45, D46, D47, D48, D49, D5, D50, D51, D52, D53, D54, D55, D56, D57, D58, D59, D6, D60, D61, D62, D63, D64, D65, D66, D67, D68, D69, D7, D70, D71, D8, D9: footprint Diode_THT:D_DO-35_SOD27_P7.62mm_Horizontal -> fortissimo-ii:D_DO-35_SOD27_P7.62mm_Horizontal
- J1, J2: footprint Keebio-Parts:TRRS-PJ-320A -> fortissimo-ii:TRRS-PJ-320A
- R1, R2, R3, R4: footprint Resistor_SMD:R_0603_1608Metric -> fortissimo-ii:R_0603_1608Metric
- SW1, SW10, SW11, SW12, SW13, SW14, SW15, SW16, SW17, SW18, SW19, SW2, SW20, SW21, SW22, SW23, SW24, SW25, SW26, SW27, SW28, SW29, SW3, SW30, SW31, SW32, SW33, SW36, SW37, SW38, SW39, SW4, SW41, SW42, SW43, SW44, SW45, SW46, SW47, SW48, SW49, SW5, SW50, SW51, SW52, SW53, SW54, SW55, SW56, SW57, SW58, SW59, SW6, SW60, SW61, SW62, SW63, SW64, SW65, SW66, SW67, SW68, SW69, SW7, SW8, SW9: footprint Keebio-Parts:Low-Profile-Choc-MX -> fortissimo-ii:Low-Profile-Choc-MX
- SW34, SW40: footprint Keebio-Parts:MX-Alps-Choc-2U-StabFlip -> fortissimo-ii:MX-Alps-Choc-2U-StabFlip
- SW35: footprint Button_Switch_THT:SW_PUSH_6mm -> fortissimo-ii:SW_PUSH_6mm
