File: _autosave-fortissimo-ii.kicad_sch (KiCad schematic)
At the start: 146 parts, among them J1 USB_A, J2 USB_A, SW1 SW_Push, SW10 SW_Push, SW11 SW_Push, SW12 SW_Push, SW13 SW_Push, SW14 SW_Push, SW15 SW_Push, SW16 SW_Push, SW17 SW_Push, SW18 SW_Push, SW19 SW_Push, SW2 SW_Push, SW20 SW_Push, SW21 SW_Push, SW22 SW_Push, SW23 SW_Push, SW24 SW_Push, SW25 SW_Push, SW26 SW_Push, SW27 SW_Push, SW28 SW_Push, SW29 SW_Push, SW3 SW_Push, SW30 SW_Push, SW31 SW_Push, SW32 SW_Push, SW33 SW_Push, SW34 SW_Push, SW35 RotaryEncoder_Switch, SW36 LANG_SWITCH, SW4 SW_Push, SW5 SW_Push, SW6 SW_Push, SW7 SW_Push, SW8 SW_Push, SW9 SW_Push, U2 FE1.1s, U3 USBLC6-2SC6, Y1 12MHz Crystal

Commit message: wired up neopixels
Connections:
- net neopixel: now reaches D67.3 (DIN)
- net neopixel: now also U1.G3 (GPIO12)
Changed lines of the file:
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@@
+		)
+	)
+	(label "neopixel"
+		(at 177.8 175.26 180)
+		(effects
+			(font
+				(size 1.27 1.27)
+			)
+			(justify right bottom)
 		)
 	)
@@
 		(effects
 			(font
+				(size 1.27 1.27)
+			)
+			(justify right bottom)
+		)
+	)
+	(label "neopixel"
+		(at 276.86 173.99 180)
+		(effects
+			(font
