File: fortissimo-ii.kicad_pcb (KiCad board)
At the start: 2 copper layers, 147.2 x 132.2 mm, 146 parts, among them J1 USB_A, J2 USB_A, SW1 SW_Push, SW10 SW_Push, SW11 SW_Push, SW12 SW_Push, SW13 SW_Push, SW14 SW_Push, SW15 SW_Push, SW16 SW_Push, SW17 SW_Push, SW18 SW_Push, SW19 SW_Push, SW2 SW_Push, SW20 SW_Push, SW21 SW_Push, SW22 SW_Push, SW23 SW_Push, SW24 SW_Push, SW25 SW_Push, SW26 SW_Push, SW27 SW_Push, SW28 SW_Push, SW29 SW_Push, SW3 SW_Push, SW30 SW_Push, SW31 SW_Push, SW32 SW_Push, SW33 SW_Push, SW34 SW_Push, SW35 RotaryEncoder_Switch, SW36 LANG_SWITCH, SW4 SW_Push, SW5 SW_Push, SW6 SW_Push, SW7 SW_Push, SW8 SW_Push, SW9 SW_Push, U2 FE1.1s, U3 USBLC6-2SC6, Y1 12MHz Crystal

Commit message: finished left side!
Routing:
- net GND: track 14.4 -> 690.4 mm, vias 0 -> 47
- net VBUS: track 1053.8 -> 1160.0 mm, vias 63 -> 69
- net /col6: track 124.2 -> 159.0 mm
- net Net-(D14-A): track 8.58 -> 12.0 mm
- net Net-(D20-A): track 8.83 -> 11.6 mm
- net /row1: track 233.1 -> 231.2 mm
- net (no net): vias 0 -> 1
- added copper zone on B.Cu, net GND
- added copper zone on F.Cu, net GND
Other:
- board size 147.2 x 132.2 mm -> 148.2 x 136.4 mm

Commit message: changes from jul 29
Parts:
- removed 0.1uF1, 0.1uF2: USB_C_Plug_USB2.0, Connector_USB:USB_C_Receptacle_JAE_DX07S016JA1R1500
- removed C1, C10, C2, C3, C4, C6: 10uF, Capacitor_SMD:C_0805_2012Metric
- removed C11, C14, C17, C20, C23: 100uF, Capacitor_SMD:C_0805_2012Metric
- removed C12, C13, C15, C16, C18, C19, C21, C22, C24, C25: 4.7nF, Capacitor_SMD:C_0805_2012Metric
- removed C5: 0.1uF, Capacitor_SMD:C_0805_2012Metric
- removed FB1: FerriteBead, Inductor_SMD:L_0805_2012Metric
- removed R6, R7: 5.1k, Resistor_SMD:R_0805_2012Metric
- removed SW_BOOTSEL1: BOOTSEL_SWITCH, Button_Switch_THT:SW_PUSH_6mm
- removed U1: ~, PGA2040:PGA2040
- removed U2: FE1.1s, Package_SO:SSOP-28_3.9x9.9mm_P0.635mm
- removed U3: USBLC6-2SC6, Package_TO_SOT_SMD:SOT-23-6
- removed Y1: 12MHz Crystal, Crystal:Crystal_SMD_3225-4Pin_3.2x2.5mm_HandSoldering
- added A1: RaspberryPi_Pico, Module:RaspberryPi_Pico_Common_Unspecified, F.Cu at (182.7, 49.2)
- added A2: RaspberryPi_Pico, Module:RaspberryPi_Pico_Common_Unspecified, F.Cu at (220.8, 49.2)
- added Brd2: SSD1306, SSD1306:128x64OLED, F.Cu at (221.1, 67.6)
- added R2: 4.7k, Resistor_SMD:R_0603_1608Metric, B.Cu at (188.1, 44.4)
- added R3: 4.7k, Resistor_SMD:R_0603_1608Metric, B.Cu at (226.3, 39.1)
- added R4: 4.7k, Resistor_SMD:R_0603_1608Metric, B.Cu at (226.5, 44.5)
- added SW37: SW_Push_45deg, Keebio-Parts:Low-Profile-Choc-MX, F.Cu at (245.3, 52.4)
- added SW38: SW_Push_45deg, Keebio-Parts:Low-Profile-Choc-MX, F.Cu at (245.3, 71.4)
- added SW39: SW_Push_45deg, Keebio-Parts:Low-Profile-Choc-MX, F.Cu at (245.3, 90.5)
- added SW40: SW_Push_45deg, Keebio-Parts:MX-Alps-Choc-2U-StabFlip, F.Cu at (254.8, 109.5)
- added SW41: SW_Push_45deg, Keebio-Parts:Low-Profile-Choc-MX, F.Cu at (264.3, 33.3)
- added SW42: SW_Push_45deg, Keebio-Parts:Low-Profile-Choc-MX, F.Cu at (264.3, 52.4)
- added SW43: SW_Push_45deg, Keebio-Parts:Low-Profile-Choc-MX, F.Cu at (264.3, 71.4)
- added SW44: SW_Push_45deg, Keebio-Parts:Low-Profile-Choc-MX, F.Cu at (264.3, 90.5)
- added SW45: SW_Push_45deg, Keebio-Parts:Low-Profile-Choc-MX, F.Cu at (283.4, 109.5)
- added SW46: SW_Push_45deg, Keebio-Parts:Low-Profile-Choc-MX, F.Cu at (283.4, 33.3)
- added SW47: SW_Push_45deg, Keebio-Parts:Low-Profile-Choc-MX, F.Cu at (283.4, 52.4)
- added SW48: SW_Push_45deg, Keebio-Parts:Low-Profile-Choc-MX, F.Cu at (283.4, 71.4)
- added SW49: SW_Push_45deg, Keebio-Parts:Low-Profile-Choc-MX, F.Cu at (283.4, 90.5)
- added SW50: SW_Push_45deg, Keebio-Parts:Low-Profile-Choc-MX, F.Cu at (302.4, 109.5)
- added SW51: SW_Push_45deg, Keebio-Parts:Low-Profile-Choc-MX, F.Cu at (302.4, 33.3)
- added SW52: SW_Push_45deg, Keebio-Parts:Low-Profile-Choc-MX, F.Cu at (302.4, 52.4)
- added SW53: SW_Push_45deg, Keebio-Parts:Low-Profile-Choc-MX, F.Cu at (302.4, 71.4)
- added SW54: SW_Push_45deg, Keebio-Parts:Low-Profile-Choc-MX, F.Cu at (302.4, 90.5)
- added SW55: SW_Push_45deg, Keebio-Parts:Low-Profile-Choc-MX, F.Cu at (321.5, 109.5)
- added SW56: SW_Push_45deg, Keebio-Parts:Low-Profile-Choc-MX, F.Cu at (321.5, 33.3)
- added SW57: SW_Push_45deg, Keebio-Parts:Low-Profile-Choc-MX, F.Cu at (321.5, 52.4)
- added SW58: SW_Push_45deg, Keebio-Parts:Low-Profile-Choc-MX, F.Cu at (321.5, 71.4)
- added SW59: SW_Push_45deg, Keebio-Parts:Low-Profile-Choc-MX, F.Cu at (321.5, 90.5)
- added SW60: SW_Push_45deg, Keebio-Parts:Low-Profile-Choc-MX, F.Cu at (340.5, 109.5)
- added SW61: SW_Push_45deg, Keebio-Parts:Low-Profile-Choc-MX, F.Cu at (340.5, 33.3)
- added SW62: SW_Push_45deg, Keebio-Parts:Low-Profile-Choc-MX, F.Cu at (340.5, 52.4)
- added SW63: SW_Push_45deg, Keebio-Parts:Low-Profile-Choc-MX, F.Cu at (340.5, 71.4)
- added SW64: SW_Push_45deg, Keebio-Parts:Low-Profile-Choc-MX, F.Cu at (340.5, 90.5)
- added SW65: SW_Push_45deg, Keebio-Parts:Low-Profile-Choc-MX, F.Cu at (359.6, 109.5)
- added SW66: SW_Push_45deg, Keebio-Parts:Low-Profile-Choc-MX, F.Cu at (359.6, 33.3)
- added SW67: SW_Push_45deg, Keebio-Parts:Low-Profile-Choc-MX, F.Cu at (359.6, 52.4)
- added SW68: SW_Push_45deg, Keebio-Parts:Low-Profile-Choc-MX, F.Cu at (359.6, 71.4)
- added SW69: SW_Push_45deg, Keebio-Parts:Low-Profile-Choc-MX, F.Cu at (359.6, 90.5)
- D1, D10, D11, D12, D13, D14, D15, D16, D17, D18, D19, D2, D20, D21, D22, D23, D24, D25, D26, D27, D28, D29, D3, D30, D31, D32, D33, D34, D4, D5, D6, D7, D8, D9: moved to B.Cu
- D35, D36, D37, D74: value D_Schottky 100uF -> PESD5V0S1UL; footprint Capacitor_THT:C_Radial_D5.0mm_H11.0mm_P2.00mm -> Diode_SMD:D_SOD-882
- D38: value D_Schottky 100uF -> D; footprint Capacitor_THT:C_Radial_D5.0mm_H11.0mm_P2.00mm -> Diode_THT:D_DO-35_SOD27_P7.62mm_Horizontal
- D39, D40, D41, D42, D43, D44, D45, D46, D47, D48, D49, D50, D51, D52, D53, D54, D55, D56, D57, D58, D59, D60, D61, D62, D63, D64, D65, D66, D67, D68, D69, D70, D71: value SK6812MINI -> D; footprint Keebio-Parts:SK6812-MINI-E -> Diode_THT:D_DO-35_SOD27_P7.62mm_Horizontal; moved to F.Cu
- D72, D73: value SK6812MINI -> PESD5V0S1UL; footprint Keebio-Parts:SK6812-MINI-E -> Diode_SMD:D_SOD-882; moved to F.Cu
- J1, J2: value USB_A -> AudioJack4; footprint Connector_USB:USB_A_Receptacle_GCT_USB1046 -> Keebio-Parts:TRRS-PJ-320A
- R1: value 2.7k -> 4.7k; footprint Resistor_SMD:R_0805_2012Metric -> Resistor_SMD:R_0603_1608Metric; moved to B.Cu
- SW1, SW10, SW11, SW12, SW13, SW14, SW15, SW16, SW17, SW18, SW19, SW2, SW20, SW21, SW22, SW23, SW24, SW25, SW26, SW27, SW28, SW29, SW3, SW30, SW31, SW32, SW33, SW4, SW5, SW6, SW7, SW8, SW9: value SW_Push -> SW_Push_45deg; footprint Keebio-Parts:MX-Alps-Choc-1U -> Keebio-Parts:Low-Profile-Choc-MX
- SW34: value SW_Push -> SW_Push_45deg; footprint Keebio-Parts:MX-Alps-Choc-1U -> Keebio-Parts:MX-Alps-Choc-2U-StabFlip
- SW35: value RotaryEncoder_Switch -> LANG; footprint Rotary_Encoder:RotaryEncoder_Alps_EC11E-Switch_Vertical_H20mm_CircularMountingHoles -> Button_Switch_THT:SW_PUSH_6mm
- SW36: value LANG_SWITCH -> SW_Push_45deg; footprint Button_Switch_THT:SW_PUSH_6mm -> Keebio-Parts:Low-Profile-Choc-MX
- moved D59 277.3 mm to (331.0, 61.9), turned to 90 degrees
- moved D71 275.8 mm to (369.1, 100.0), turned to 90 degrees
- moved D60 273.9 mm to (331.0, 81.0), turned to 90 degrees
- moved D58 262.5 mm to (331.0, 42.9), turned to 90 degrees
- moved D62 256.9 mm to (350.0, 119.1), turned to 90 degrees
- moved D61 255.1 mm to (331.0, 100.0), turned to 90 degrees
- moved D70 255.0 mm to (369.1, 81.0), turned to 90 degrees
- moved D63 239.9 mm to (350.0, 42.9), turned to 90 degrees
- moved D57 236.2 mm to (331.0, 119.1), turned to 90 degrees
- moved D69 235.8 mm to (369.1, 61.9), turned to 90 degrees
- moved D68 218.1 mm to (369.1, 42.9), turned to 90 degrees
- moved D64 218.1 mm to (350.0, 61.9), turned to 90 degrees
- moved D46 218.1 mm to (273.8, 100.0), turned to 90 degrees
- moved D47 216.8 mm to (292.9, 119.1), turned to 90 degrees
- moved D39 214.1 mm to (254.8, 61.9), turned to 90 degrees
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Connections:
- net /col1 renamed /L_col_1
- net /col2 renamed /L_col_2
- net /col3 renamed /L_col_3
- net /col4 renamed /L_col_4
- net /col5 renamed /L_col_5
- net /col6 renamed /L_col_6
- net /col7 renamed /L_col_7
- net /row1 renamed /L_row_1
- net /row2 renamed /L_row_2
- net /row3 renamed /L_row_3
- net /row4 renamed /L_row_4
- net /row5 renamed /L_row_5
- Brd1 pad 2: +3.3V -> VBUS
- Brd1 pad 3: Net-(Brd1-SCL) -> /L_SCL
- Brd1 pad 4: Net-(Brd1-SDA) -> /L_SDA
- D35 pad 1: Net-(D35-K) -> GND
- D35 pad 2: Net-(D35-A) -> VBUS
- D36 pad 1: Net-(D36-K) -> GND
- D36 pad 2: VBUS -> /L_SDA
- D37 pad 1: Net-(D37-K) -> GND
- D37 pad 2: VBUS -> /L_SCL
- D38 pad 1: Net-(D38-K) -> /R_row_1
- D38 pad 2: VBUS -> Net-(D38-A)
- D39 pad 1: unconnected-(D39-DOUT-Pad1) -> /R_row_2
- D39 pad 2: GND -> Net-(D39-A)
- D40 pad 1: Net-(D39-DIN) -> /R_row_3
- D40 pad 2: GND -> Net-(D40-A)
- D41 pad 1: Net-(D40-DIN) -> /R_row_4
- D41 pad 2: GND -> Net-(D41-A)
- D42 pad 1: Net-(D41-DIN) -> /R_row_5
- D42 pad 2: GND -> Net-(D42-A)
- D43 pad 1: Net-(D42-DIN) -> /R_row_1
- D43 pad 2: GND -> Net-(D43-A)
- D44 pad 1: Net-(D43-DIN) -> /R_row_2
- D44 pad 2: GND -> Net-(D44-A)
- D45 pad 1: Net-(D44-DIN) -> /R_row_3
- D45 pad 2: GND -> Net-(D45-A)
- D46 pad 1: Net-(D46-DOUT) -> /R_row_4
- D46 pad 2: GND -> Net-(D46-A)
- D47 pad 1: Net-(D47-DOUT) -> /R_row_5
- D47 pad 2: GND -> Net-(D47-A)
- D48 pad 1: Net-(D48-DOUT) -> /R_row_1
- D48 pad 2: GND -> Net-(D48-A)
- D49 pad 1: Net-(D49-DOUT) -> /R_row_2
- D49 pad 2: GND -> Net-(D49-A)
- D50 pad 1: Net-(D50-DOUT) -> /R_row_3
- D50 pad 2: GND -> Net-(D50-A)
- D51 pad 1: Net-(D51-DOUT) -> /R_row_4
- D51 pad 2: GND -> Net-(D51-A)
- D52 pad 1: Net-(D45-DIN) -> /R_row_5
- D52 pad 2: GND -> Net-(D52-A)
- D53 pad 1: Net-(D53-DOUT) -> /R_row_1
- D53 pad 2: GND -> Net-(D53-A)
- D54 pad 1: Net-(D54-DOUT) -> /R_row_2
- D54 pad 2: GND -> Net-(D54-A)
- D55 pad 1: Net-(D55-DOUT) -> /R_row_3
- D55 pad 2: GND -> Net-(D55-A)
- D56 pad 1: Net-(D56-DOUT) -> /R_row_4
- D56 pad 2: GND -> Net-(D56-A)
- D57 pad 1: Net-(D57-DOUT) -> /R_row_5
- D57 pad 2: GND -> Net-(D57-A)
- D58 pad 1: Net-(D58-DOUT) -> /R_row_1
- D58 pad 2: GND -> Net-(D58-A)
- D59 pad 1: Net-(D46-DIN) -> /R_row_2
- D59 pad 2: GND -> Net-(D59-A)
- D60 pad 1: Net-(D60-DOUT) -> /R_row_3
- D60 pad 2: GND -> Net-(D60-A)
- D61 pad 1: Net-(D61-DOUT) -> /R_row_4
- D61 pad 2: GND -> Net-(D61-A)
- D62 pad 1: Net-(D62-DOUT) -> /R_row_5
- D62 pad 2: GND -> Net-(D62-A)
- D63 pad 1: Net-(D63-DOUT) -> /R_row_1
- D63 pad 2: GND -> Net-(D63-A)
- D64 pad 1: Net-(D64-DOUT) -> /R_row_2
- D64 pad 2: GND -> Net-(D64-A)
- D65 pad 1: Net-(D65-DOUT) -> /R_row_3
- D65 pad 2: GND -> Net-(D65-A)
- D66 pad 1: Net-(D53-DIN) -> /R_row_4
- D66 pad 2: GND -> Net-(D66-A)
- D67 pad 1: Net-(D67-DOUT) -> /R_row_5
- D67 pad 2: GND -> Net-(D67-A)
- D68 pad 1: Net-(D68-DOUT) -> /R_row_1
- D68 pad 2: GND -> Net-(D68-A)
- D69 pad 1: Net-(D69-DOUT) -> /R_row_2
- D69 pad 2: GND -> Net-(D69-A)
- D70 pad 1: Net-(D70-DOUT) -> /R_row_3
- D70 pad 2: GND -> Net-(D70-A)
- D71 pad 1: Net-(D71-DOUT) -> /R_row_4
- D71 pad 2: GND -> Net-(D71-A)
- D72 pad 1: Net-(D72-DOUT) -> GND
- D72 pad 2: GND -> VBUS
- D73 pad 1: Net-(D60-DIN) -> GND
- D73 pad 2: GND -> /R_SDA
- D74 pad 1: Net-(D74-K) -> GND
- D74 pad 2: VBUS -> /R_SCL
- R1 pad 1: GND -> VBUS
- R1 pad 2: Net-(U2-REXT) -> /L_SDA
- SW36 pad 1: /LANG -> /R_col_1
- SW36 pad 2: GND -> Net-(D38-A)
Routing:
- net VBUS: track 1160.0 -> 141.8 mm, vias 69 -> 6
- net GND: track 690.4 -> 0.57 mm, vias 47 -> 0
- net /R_col_7: track 0.00 -> 246.6 mm, vias 0 -> 2
- net /R_col_6: track 0.00 -> 228.3 mm, vias 0 -> 2
- net /R_col_5: track 0.00 -> 217.2 mm, vias 0 -> 2
- net /R_row_4: track 0.00 -> 213.8 mm, vias 0 -> 1
- net /R_col_4: track 0.00 -> 197.1 mm, vias 0 -> 2
- net /R_col_3: track 0.00 -> 176.4 mm, vias 0 -> 2
- net /R_row_1: track 0.00 -> 164.6 mm, vias 0 -> 1
- net /R_col_2: track 0.00 -> 146.1 mm, vias 0 -> 2
- net /R_row_5: track 0.00 -> 129.6 mm, vias 0 -> 1
- net Net-(J1-D+): track 125.3 -> 0.00 mm
- net Net-(U1-BOOTSEL): track 123.2 -> 0.00 mm
- net Net-(J1-D-): track 123.2 -> 0.00 mm
- net /R_col_1: track 0.00 -> 119.8 mm
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- removed copper zone on B.Cu, net GND
Other:
- board size 148.2 x 136.4 mm -> 341.8 x 98.7 mm

Commit message: basically the entire thing
Parts:
- added REF**: MountingHole_3.2mm_M3, MountingHole:MountingHole_3.2mm_M3, F.Cu at (376.2, 71.9)
- added REF**: MountingHole_3.2mm_M3, MountingHole:MountingHole_3.2mm_M3, F.Cu at (190.5, 117.5)
- added REF**: MountingHole_3.2mm_M3, MountingHole:MountingHole_3.2mm_M3, F.Cu at (211.9, 117.5)
- added REF**: MountingHole_3.2mm_M3, MountingHole:MountingHole_3.2mm_M3, F.Cu at (178.6, 100.0)
- added REF**: MountingHole_3.2mm_M3, MountingHole:MountingHole_3.2mm_M3, F.Cu at (376.2, 26.2)
- added REF**: MountingHole_3.2mm_M3, MountingHole:MountingHole_3.2mm_M3, F.Cu at (28.6, 116.7)
- added REF**: MountingHole_3.2mm_M3, MountingHole:MountingHole_3.2mm_M3, F.Cu at (28.6, 71.4)
- added REF**: MountingHole_3.2mm_M3, MountingHole:MountingHole_3.2mm_M3, F.Cu at (376.2, 116.7)
- added REF**: MountingHole_3.2mm_M3, MountingHole:MountingHole_3.2mm_M3, F.Cu at (226.2, 100.0)
- added REF**: MountingHole_3.2mm_M3, MountingHole:MountingHole_3.2mm_M3, F.Cu at (28.6, 26.2)
- A1, A2: footprint Module:RaspberryPi_Pico_Common_Unspecified -> fortissimo-ii:RaspberryPi_Pico_Common_Unspecified
- Brd1, Brd2: footprint SSD1306:128x64OLED -> fortissimo-ii:128x64OLED
- D1, D10, D11, D12, D13, D14, D15, D16, D17, D18, D19, D2, D20, D21, D22, D23, D24, D25, D26, D27, D28, D29, D3, D30, D31, D32, D33, D34, D4, D5, D6, D7, D8, D9: footprint Diode_THT:D_DO-35_SOD27_P7.62mm_Horizontal -> fortissimo-ii:D_DO-35_SOD27_P7.62mm_Horizontal
- D38, D39, D40, D41, D42, D43, D44, D45, D46, D47, D48, D49, D50, D51, D52, D53, D54, D55, D56, D57, D58, D59, D60, D61, D62, D63, D64, D65, D66, D67, D68, D69, D70, D71: footprint Diode_THT:D_DO-35_SOD27_P7.62mm_Horizontal -> fortissimo-ii:D_DO-35_SOD27_P7.62mm_Horizontal; moved to B.Cu
- J1, J2: footprint Keebio-Parts:TRRS-PJ-320A -> fortissimo-ii:TRRS-PJ-320A
- R1, R2, R3, R4: footprint Resistor_SMD:R_0603_1608Metric -> fortissimo-ii:R_0603_1608Metric
- SW1, SW10, SW11, SW12, SW13, SW14, SW15, SW16, SW17, SW18, SW19, SW2, SW20, SW21, SW22, SW23, SW24, SW25, SW26, SW27, SW28, SW29, SW3, SW30, SW31, SW32, SW33, SW36, SW37, SW38, SW39, SW4, SW41, SW42, SW43, SW44, SW45, SW46, SW47, SW48, SW49, SW5, SW50, SW51, SW52, SW53, SW54, SW55, SW56, SW57, SW58, SW59, SW6, SW60, SW61, SW62, SW63, SW64, SW65, SW66, SW67, SW68, SW69, SW7, SW8, SW9: footprint Keebio-Parts:Low-Profile-Choc-MX -> fortissimo-ii:Low-Profile-Choc-MX
- SW34, SW40: footprint Keebio-Parts:MX-Alps-Choc-2U-StabFlip -> fortissimo-ii:MX-Alps-Choc-2U-StabFlip
- SW35: footprint Button_Switch_THT:SW_PUSH_6mm -> fortissimo-ii:SW_PUSH_6mm
- moved D72 4.02 mm to (223.5, 95.2)
- moved D36 2.36 mm to (191.1, 100.1)
- moved D37 2.36 mm to (188.1, 100.2)
- moved J1 2.22 mm to (194.5, 95.3)
- moved D35 2.13 mm to (180.6, 93.0)
- moved D73 1.75 mm to (211.3, 90.2)
- moved D74 1.75 mm to (214.3, 90.3)
- moved J2 1.60 mm to (207.9, 95.3)
- moved Brd1 1.32 mm to (181.5, 67.6)
- moved Brd2 0.41 mm to (221.5, 67.6)
Routing:
- net VBUS: track 141.8 -> 162.7 mm
- net Net-(D55-A): track 0.00 -> 19.3 mm
- net Net-(D70-A): track 0.00 -> 19.3 mm
- net Net-(D65-A): track 0.00 -> 19.3 mm
- net Net-(D60-A): track 0.00 -> 19.3 mm
- net /L_SCL: track 66.8 -> 64.9 mm
- net GND: track 0.57 -> 0.00 mm
Other:
- board size 341.8 x 98.7 mm -> 357.2 x 100 mm
- board text added: "fortissimo"
- board text added: "gbtsui"
